File: ppuppy/pcb/realbreakout/realbreakout.kicad_pcb (KiCad board)
At the start: 2 copper layers, 99.6 x 88.6 mm, 24 parts, among them J1 Conn_01x36, J10 BCM11, J11 BCM13, J12 /OE, J2 Conn_01x36, J3 Conn_01x36, J4 BCM25, J5 BCM24, J6 BCM27, J7 3V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

Commit message: Cart plays sound for debugging when video is not present. Fix circuit board layout
Parts:
- .1uf1, .1uf2, .1uf3: value .1uf -> C
Connections:
- .1uf1 pad 2: 5V -> 5v
- E1 pad 31: GND -> 5v
- E1 pad 32: 5V -> 5v
- J1 pad 36: 5V -> 5v
- J2 pad 16: 5V -> 5v
- J3 pad 16: 5V -> 5v
- U1 pad 36: 5V -> 5v
- U1 pad 57: 5V -> 5v
- U2 pad 2: 5V -> 5v
- U2 pad 4: 5V -> 5v
- U3 pad 16: 5V -> 5v
- U4 pad 20: 5V -> 5v
Routing:
- net 5v: track 0.00 -> 330.7 mm
- net 5V: track 328.2 -> 0.00 mm
Other:
- board text added: "v3!"
- board text removed: "v2!"
